Commit message: moved working model to "hexapod" pkg

File: src/hexapod/urdf/robot.urdf.xacro (robot description, xacro)
@@ -1,6 +1,6 @@
 <?xml version="1.0"?>
 <robot name="my_robot" xmlns:xacro="http://www.ros.org/wiki/xacro">
-	<xacro:include filename="$(find my_robot_description)/urdf/materials.xacro" />
-  <xacro:include filename="$(find my_robot_description)/urdf/robot.gazebo.xacro"/>
+	<xacro:include filename="$(find hexapod)/urdf/materials.xacro" />
+  <xacro:include filename="$(find hexapod)/urdf/robot.gazebo.xacro"/>
   <gazebo>
         <self_collide>1</self_collide>
@@ -21,5 +21,5 @@
       <origin rpy="0 0 0" xyz="0.4 -0.75 -0.115"/>
       <geometry>
-        <mesh filename="package://my_robot_description/model/stl/Body.stl" scale="0.01 0.01 0.01"/>
+        <mesh filename="package://hexapod/model/stl/Body.stl" scale="0.01 0.01 0.01"/>
       </geometry>
     </collision>
@@ -27,5 +27,5 @@
       <origin rpy="0 0 0" xyz="0.4 -0.75 -0.115"/>
       <geometry>
-        <mesh filename="package://my_robot_description/model/stl/Body.stl" scale="0.01 0.01 0.01"/>
+        <mesh filename="package://hexapod/model/stl/Body.stl" scale="0.01 0.01 0.01"/>
       </geometry>
       <material name="white"/>
@@ -45,5 +45,5 @@
       <origin rpy="0 0 0" xyz="0.4 -0.75 -0.115"/>
       <geometry>
-        <mesh filename="package://my_robot_description/model/stl/Body.stl" scale="0.01 0.01 0.01"/>
+        <mesh filename="package://hexapod/model/stl/Body.stl" scale="0.01 0.01 0.01"/>
       </geometry>
     </collision>
@@ -51,5 +51,5 @@
       <origin rpy="0 0 0" xyz="0.4 -0.75 -0.115"/>
       <geometry>
-        <mesh filename="package://my_robot_description/model/stl/Body.stl" scale="0.01 0.01 0.01"/>
+        <mesh filename="package://hexapod/model/stl/Body.stl" scale="0.01 0.01 0.01"/>
       </geometry>
       <material name="white"/>
@@ -69,11 +69,11 @@
       <origin rpy="0 0 0" xyz="-0.06 -0.1125 -0.164"/>
       <geometry>
-        <mesh filename="package://my_robot_description/model/stl/ServoMG90S.stl" scale="0.01 0.01 0.01"/>
-      </geometry>
-    </collision>
-    <visual>
-      <origin rpy="0 0 0" xyz="-0.06 -0.1125 -0.164"/>
-      <geometry>
-        <mesh filename="package://my_robot_description/model/stl/ServoMG90S.stl" scale="0.01 0.01 0.01"/>
+        <mesh filename="package://hexapod/model/stl/ServoMG90S.stl" scale="0.01 0.01 0.01"/>
+      </geometry>
+    </collision>
+    <visual>
+      <origin rpy="0 0 0" xyz="-0.06 -0.1125 -0.164"/>
+      <geometry>
+        <mesh filename="package://hexapod/model/stl/ServoMG90S.stl" scale="0.01 0.01 0.01"/>
       </geometry>
       <material name="light_black"/>
@@ -93,11 +93,11 @@
       <origin rpy="0 0 0" xyz="-0.06 -0.1125 -0.164"/>
       <geometry>
-        <mesh filename="package://my_robot_description/model/stl/ServoMG90S.stl" scale="0.01 0.01 0.01"/>
-      </geometry>
-    </collision>
-    <visual>
-      <origin rpy="0 0 0" xyz="-0.06 -0.1125 -0.164"/>
-      <geometry>
-        <mesh filename="package://my_robot_description/model/stl/ServoMG90S.stl" scale="0.01 0.01 0.01"/>
+        <mesh filename="package://hexapod/model/stl/ServoMG90S.stl" scale="0.01 0.01 0.01"/>
+      </geometry>
+    </collision>
+    <visual>
+      <origin rpy="0 0 0" xyz="-0.06 -0.1125 -0.164"/>
+      <geometry>
+        <mesh filename="package://hexapod/model/stl/ServoMG90S.stl" scale="0.01 0.01 0.01"/>
       </geometry>
       <material name="light_black"/>
@@ -117,11 +117,11 @@
       <origin rpy="0 0 0" xyz="-0.06 -0.1125 -0.164"/>
       <geometry>
-        <mesh filename="package://my_robot_description/model/stl/ServoMG90S.stl" scale="0.01 0.01 0.01"/>
-      </geometry>
-    </collision>
-    <visual>
-      <origin rpy="0 0 0" xyz="-0.06 -0.1125 -0.164"/>
-      <geometry>
-        <mesh filename="package://my_robot_description/model/stl/ServoMG90S.stl" scale="0.01 0.01 0.01"/>
+        <mesh filename="package://hexapod/model/stl/ServoMG90S.stl" scale="0.01 0.01 0.01"/>
+      </geometry>
+    </collision>
+    <visual>
+      <origin rpy="0 0 0" xyz="-0.06 -0.1125 -0.164"/>
+      <geometry>
+        <mesh filename="package://hexapod/model/stl/ServoMG90S.stl" scale="0.01 0.01 0.01"/>
       </geometry>
       <material name="light_black"/>
@@ -141,11 +141,11 @@
       <origin rpy="0 0 0" xyz="-0.06 -0.1125 -0.164"/>
       <geometry>
-        <mesh filename="package://my_robot_description/model/stl/ServoMG90S.stl" scale="0.01 0.01 0.01"/>
-      </geometry>
-    </collision>
-    <visual>
-      <origin rpy="0 0 0" xyz="-0.06 -0.1125 -0.164"/>
-      <geometry>
-        <mesh filename="package://my_robot_description/model/stl/ServoMG90S.stl" scale="0.01 0.01 0.01"/>
+        <mesh filename="package://hexapod/model/stl/ServoMG90S.stl" scale="0.01 0.01 0.01"/>
+      </geometry>
+    </collision>
+    <visual>
+      <origin rpy="0 0 0" xyz="-0.06 -0.1125 -0.164"/>
+      <geometry>
+        <mesh filename="package://hexapod/model/stl/ServoMG90S.stl" scale="0.01 0.01 0.01"/>
       </geometry>
       <material name="light_black"/>
@@ -165,11 +165,11 @@
       <origin rpy="0 0 0" xyz="-0.06 -0.1125 -0.164"/>
       <geometry>
-        <mesh filename="package://my_robot_description/model/stl/ServoMG90S.stl" scale="0.01 0.01 0.01"/>
-      </geometry>
-    </collision>
-    <visual>
-      <origin rpy="0 0 0" xyz="-0.06 -0.1125 -0.164"/>
-      <geometry>
-        <mesh filename="package://my_robot_description/model/stl/ServoMG90S.stl" scale="0.01 0.01 0.01"/>
+        <mesh filename="package://hexapod/model/stl/ServoMG90S.stl" scale="0.01 0.01 0.01"/>
+      </geometry>
+    </collision>
+    <visual>
+      <origin rpy="0 0 0" xyz="-0.06 -0.1125 -0.164"/>
+      <geometry>
+        <mesh filename="package://hexapod/model/stl/ServoMG90S.stl" scale="0.01 0.01 0.01"/>
       </geometry>
       <material name="light_black"/>
@@ -188,11 +188,11 @@
       <origin rpy="0 0 0" xyz="-0.06 -0.1125 -0.164"/>
       <geometry>
-        <mesh filename="package://my_robot_description/model/stl/ServoMG90S.stl" scale="0.01 0.01 0.01"/>
-      </geometry>
-    </collision>
-    <visual>
-      <origin rpy="0 0 0" xyz="-0.06 -0.1125 -0.164"/>
-      <geometry>
-        <mesh filename="package://my_robot_description/model/stl/ServoMG90S.stl" scale="0.01 0.01 0.01"/>
+        <mesh filename="package://hexapod/model/stl/ServoMG90S.stl" scale="0.01 0.01 0.01"/>
+      </geometry>
+    </collision>
+    <visual>
+      <origin rpy="0 0 0" xyz="-0.06 -0.1125 -0.164"/>
+      <geometry>
+        <mesh filename="package://hexapod/model/stl/ServoMG90S.stl" scale="0.01 0.01 0.01"/>
       </geometry>
       <material name="light_black"/>
@@ -212,11 +212,11 @@
       <origin rpy="0 0 0" xyz="-0.055 -0.2343822 -0.045"/>
       <geometry>
-        <mesh filename="package://my_robot_description/model/stl/Leg_p1.stl" scale="0.01 0.01 0.01"/>
-      </geometry>
-    </collision>
-    <visual>
-      <origin rpy="0 0 0" xyz="-0.055 -0.2343822 -0.045"/>
-      <geometry>
-        <mesh filename="package://my_robot_description/model/stl/Leg_p1.stl" scale="0.01 0.01 0.01"/>
+        <mesh filename="package://hexapod/model/stl/Leg_p1.stl" scale="0.01 0.01 0.01"/>
+      </geometry>
+    </collision>
+    <visual>
+      <origin rpy="0 0 0" xyz="-0.055 -0.2343822 -0.045"/>
+      <geometry>
+        <mesh filename="package://hexapod/model/stl/Leg_p1.stl" scale="0.01 0.01 0.01"/>
       </geometry>
       <material name="white"/>
@@ -236,11 +236,11 @@
       <origin rpy="0 0 0" xyz="-0.055 -0.2343822 -0.045"/>
       <geometry>
-        <mesh filename="package://my_robot_description/model/stl/Leg_p1.stl" scale="0.01 0.01 0.01"/>
-      </geometry>
-    </collision>
-    <visual>
-      <origin rpy="0 0 0" xyz="-0.055 -0.2343822 -0.045"/>
-      <geometry>
-        <mesh filename="package://my_robot_description/model/stl/Leg_p1.stl" scale="0.01 0.01 0.01"/>
+        <mesh filename="package://hexapod/model/stl/Leg_p1.stl" scale="0.01 0.01 0.01"/>
+      </geometry>
+    </collision>
+    <visual>
+      <origin rpy="0 0 0" xyz="-0.055 -0.2343822 -0.045"/>
+      <geometry>
+        <mesh filename="package://hexapod/model/stl/Leg_p1.stl" scale="0.01 0.01 0.01"/>
       </geometry>
       <material name="white"/>
@@ -260,11 +260,11 @@
       <origin rpy="0 0 0" xyz="-0.055 -0.2343822 -0.045"/>
       <geometry>
-        <mesh filename="package://my_robot_description/model/stl/Leg_p1.stl" scale="0.01 0.01 0.01"/>
-      </geometry>
-    </collision>
-    <visual>
-      <origin rpy="0 0 0" xyz="-0.055 -0.2343822 -0.045"/>
-      <geometry>
-        <mesh filename="package://my_robot_description/model/stl/Leg_p1.stl" scale="0.01 0.01 0.01"/>
+        <mesh filename="package://hexapod/model/stl/Leg_p1.stl" scale="0.01 0.01 0.01"/>
+      </geometry>
+    </collision>
+    <visual>
+      <origin rpy="0 0 0" xyz="-0.055 -0.2343822 -0.045"/>
+      <geometry>
+        <mesh filename="package://hexapod/model/stl/Leg_p1.stl" scale="0.01 0.01 0.01"/>
       </geometry>
       <material name="white"/>
@@ -284,11 +284,11 @@
       <origin rpy="0 0 0" xyz="-0.055 -0.2343822 -0.045"/>
       <geometry>
-        <mesh filename="package://my_robot_description/model/stl/Leg_p1.stl" scale="0.01 0.01 0.01"/>
-      </geometry>
-    </collision>
-    <visual>
-      <origin rpy="0 0 0" xyz="-0.055 -0.2343822 -0.045"/>
-      <geometry>
-        <mesh filename="package://my_robot_description/model/stl/Leg_p1.stl" scale="0.01 0.01 0.01"/>
+        <mesh filename="package://hexapod/model/stl/Leg_p1.stl" scale="0.01 0.01 0.01"/>
+      </geometry>
+    </collision>
+    <visual>
+      <origin rpy="0 0 0" xyz="-0.055 -0.2343822 -0.045"/>
+      <geometry>
+        <mesh filename="package://hexapod/model/stl/Leg_p1.stl" scale="0.01 0.01 0.01"/>
       </geometry>
       <material name="white"/>
@@ -308,11 +308,11 @@
       <origin rpy="0 0 0" xyz="-0.055 -0.2343822 -0.045"/>
       <geometry>
-        <mesh filename="package://my_robot_description/model/stl/Leg_p1.stl" scale="0.01 0.01 0.01"/>
-      </geometry>
-    </collision>
-    <visual>
-      <origin rpy="0 0 0" xyz="-0.055 -0.2343822 -0.045"/>
-      <geometry>
-        <mesh filename="package://my_robot_description/model/stl/Leg_p1.stl" scale="0.01 0.01 0.01"/>
+        <mesh filename="package://hexapod/model/stl/Leg_p1.stl" scale="0.01 0.01 0.01"/>
+      </geometry>
+    </collision>
+    <visual>
+      <origin rpy="0 0 0" xyz="-0.055 -0.2343822 -0.045"/>
+      <geometry>
+        <mesh filename="package://hexapod/model/stl/Leg_p1.stl" scale="0.01 0.01 0.01"/>
       </geometry>
       <material name="white"/>
@@ -331,11 +331,11 @@
       <origin rpy="0 0 0" xyz="-0.055 -0.2343822 -0.045"/>
       <geometry>
-        <mesh filename="package://my_robot_description/model/stl/Leg_p1.stl" scale="0.01 0.01 0.01"/>
-      </geometry>
-    </collision>
-    <visual>
-      <origin rpy="0 0 0" xyz="-0.055 -0.2343822 -0.045"/>
-      <geometry>
-        <mesh filename="package://my_robot_description/model/stl/Leg_p1.stl" scale="0.01 0.01 0.01"/>
+        <mesh filename="package://hexapod/model/stl/Leg_p1.stl" scale="0.01 0.01 0.01"/>
+      </geometry>
+    </collision>
+    <visual>
+      <origin rpy="0 0 0" xyz="-0.055 -0.2343822 -0.045"/>
+      <geometry>
+        <mesh filename="package://hexapod/model/stl/Leg_p1.stl" scale="0.01 0.01 0.01"/>
       </geometry>
       <material name="white"/>
@@ -354,11 +354,11 @@
       <origin rpy="0 0 0" xyz="-0.06 ${-0.1125-0.0525} ${-0.164+0.099}"/>
       <geometry>
-        <mesh filename="package://my_robot_description/model/stl/ServoMG90S.stl" scale="0.01 0.01 0.01"/>
-      </geometry>
-    </collision>
-    <visual>
-      <origin rpy="0 0 0" xyz="-0.06 ${-0.1125-0.0525} ${-0.164+0.099}"/>
-      <geometry>
-        <mesh filename="package://my_robot_description/model/stl/ServoMG90S.stl" scale="0.01 0.01 0.01"/>
+        <mesh filename="package://hexapod/model/stl/ServoMG90S.stl" scale="0.01 0.01 0.01"/>
+      </geometry>
+    </collision>
+    <visual>
+      <origin rpy="0 0 0" xyz="-0.06 ${-0.1125-0.0525} ${-0.164+0.099}"/>
+      <geometry>
+        <mesh filename="package://hexapod/model/stl/ServoMG90S.stl" scale="0.01 0.01 0.01"/>
       </geometry>
       <material name="light_black"/>
@@ -377,11 +377,11 @@
       <origin rpy="0 0 0" xyz="-0.33 -0.115 ${-0.1041745 + 0.044}"/>
       <geometry>
-        <mesh filename="package://my_robot_description/model/stl/Leg_p2.stl" scale="0.01 0.01 0.01"/>
-      </geometry>
-    </collision>
-    <visual>
-      <origin rpy="0 0 0" xyz="-0.33 -0.115 ${-0.1041745 + 0.044}"/>
-      <geometry>
-        <mesh filename="package://my_robot_description/model/stl/Leg_p2.stl" scale="0.01 0.01 0.01"/>
+        <mesh filename="package://hexapod/model/stl/Leg_p2.stl" scale="0.01 0.01 0.01"/>
+      </geometry>
+    </collision>
+    <visual>
+      <origin rpy="0 0 0" xyz="-0.33 -0.115 ${-0.1041745 + 0.044}"/>
+      <geometry>
+        <mesh filename="package://hexapod/model/stl/Leg_p2.stl" scale="0.01 0.01 0.01"/>
       </geometry>
       <material name="orange"/>
@@ -400,11 +400,11 @@
       <origin rpy="0 0 0" xyz="-0.06 -0.1125 -0.164"/>
       <geometry>
-        <mesh filename="package://my_robot_description/model/stl/ServoMG90S.stl" scale="0.01 0.01 0.01"/>
-      </geometry>
-    </collision>
-    <visual>
-      <origin rpy="0 0 0" xyz="-0.06 -0.1125 -0.164"/>
-      <geometry>
-        <mesh filename="package://my_robot_description/model/stl/ServoMG90S.stl" scale="0.01 0.01 0.01"/>
+        <mesh filename="package://hexapod/model/stl/ServoMG90S.stl" scale="0.01 0.01 0.01"/>
+      </geometry>
+    </collision>
+    <visual>
+      <origin rpy="0 0 0" xyz="-0.06 -0.1125 -0.164"/>
+      <geometry>
+        <mesh filename="package://hexapod/model/stl/ServoMG90S.stl" scale="0.01 0.01 0.01"/>
       </geometry>
       <material name="light_black"/>
@@ -423,11 +423,11 @@
       <origin rpy="0 0 0" xyz="${-0.2-0.065} 0 ${0.2041745-0.3591745}"/>
       <geometry>
-        <mesh filename="package://my_robot_description/model/stl/Leg_p3.stl" scale="0.01 0.01 0.01"/>
-      </geometry>
-    </collision>
-    <visual>
-      <origin rpy="0 0 0" xyz="${-0.2-0.065} 0 ${0.2041745-0.3591745}"/>
-      <geometry>
-        <mesh filename="package://my_robot_description/model/stl/Leg_p3.stl" scale="0.01 0.01 0.01"/>
+        <mesh filename="package://hexapod/model/stl/Leg_p3.stl" scale="0.01 0.01 0.01"/>
+      </geometry>
+    </collision>
+    <visual>
+      <origin rpy="0 0 0" xyz="${-0.2-0.065} 0 ${0.2041745-0.3591745}"/>
+      <geometry>
+        <mesh filename="package://hexapod/model/stl/Leg_p3.stl" scale="0.01 0.01 0.01"/>
       </geometry>
       <material name="white"/>
@@ -446,11 +446,11 @@
       <origin rpy="0 0 0" xyz="-0.06 ${-0.1125-0.0525} ${-0.164+0.099}"/>
       <geometry>
-        <mesh filename="package://my_robot_description/model/stl/ServoMG90S.stl" scale="0.01 0.01 0.01"/>
-      </geometry>
-    </collision>
-    <visual>
-      <origin rpy="0 0 0" xyz="-0.06 ${-0.1125-0.0525} ${-0.164+0.099}"/>
-      <geometry>
-        <mesh filename="package://my_robot_description/model/stl/ServoMG90S.stl" scale="0.01 0.01 0.01"/>
+        <mesh filename="package://hexapod/model/stl/ServoMG90S.stl" scale="0.01 0.01 0.01"/>
+      </geometry>
+    </collision>
+    <visual>
+      <origin rpy="0 0 0" xyz="-0.06 ${-0.1125-0.0525} ${-0.164+0.099}"/>
+      <geometry>
+        <mesh filename="package://hexapod/model/stl/ServoMG90S.stl" scale="0.01 0.01 0.01"/>
       </geometry>
       <material name="light_black"/>
@@ -469,11 +469,11 @@
       <origin rpy="0 0 0" xyz="-0.33 -0.115 ${-0.1041745 + 0.044}"/>
       <geometry>
-        <mesh filename="package://my_robot_description/model/stl/Leg_p2.stl" scale="0.01 0.01 0.01"/>
-      </geometry>
-    </collision>
-    <visual>
-      <origin rpy="0 0 0" xyz="-0.33 -0.115 ${-0.1041745 + 0.044}"/>
-      <geometry>
-        <mesh filename="package://my_robot_description/model/stl/Leg_p2.stl" scale="0.01 0.01 0.01"/>
+        <mesh filename="package://hexapod/model/stl/Leg_p2.stl" scale="0.01 0.01 0.01"/>
+      </geometry>
+    </collision>
+    <visual>
+      <origin rpy="0 0 0" xyz="-0.33 -0.115 ${-0.1041745 + 0.044}"/>
+      <geometry>
+        <mesh filename="package://hexapod/model/stl/Leg_p2.stl" scale="0.01 0.01 0.01"/>
       </geometry>
       <material name="orange"/>
@@ -492,11 +492,11 @@
       <origin rpy="0 0 0" xyz="-0.06 -0.1125 -0.164"/>
       <geometry>
-        <mesh filename="package://my_robot_description/model/stl/ServoMG90S.stl" scale="0.01 0.01 0.01"/>
-      </geometry>
-    </collision>
-    <visual>
-      <origin rpy="0 0 0" xyz="-0.06 -0.1125 -0.164"/>
-      <geometry>
-        <mesh filename="package://my_robot_description/model/stl/ServoMG90S.stl" scale="0.01 0.01 0.01"/>
+        <mesh filename="package://hexapod/model/stl/ServoMG90S.stl" scale="0.01 0.01 0.01"/>
+      </geometry>
+    </collision>
+    <visual>
+      <origin rpy="0 0 0" xyz="-0.06 -0.1125 -0.164"/>
+      <geometry>
+        <mesh filename="package://hexapod/model/stl/ServoMG90S.stl" scale="0.01 0.01 0.01"/>
       </geometry>
       <material name="light_black"/>
@@ -515,11 +515,11 @@
       <origin rpy="0 0 0" xyz="${-0.2-0.065} 0 ${0.2041745-0.3591745}"/>
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